Commit message: Added Maze2 World for testing

File: path_planning_ws/src/maze_bot/urdf/maze_bot.urdf (robot description, URDF)
Before this commit: robot maze_bot, 5 links, 4 joints
Links:
- added link camera_link
Joints:
- added joint camera_joint: type fixed, parent base, child camera_link, origin xyz=-0.16 0.0 0.08 rpy=0 0.0 3.14, axis 0.0 0.0 1.0
